File: negL/ball_breakout/ball_breakout.kicad_sch (KiCad schematic)
At the start: 14 parts, among them J1 XA-3-2-7P Contact, U1 PAW3395, U2 VRH1902LTX

Commit message: Add switches
Parts:
- U1: now left out of the parts list
Changed lines of the file:
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@@
 		(unit 1)
 		(exclude_from_sim no)
-		(in_bom yes)
+		(in_bom no)
 		(on_board yes)
 		(dnp no)

Commit message: update
Parts:
- removed C8: CC0603KRX7R9BB104, Capacitor_SMD:C_0603_1608Metric, symbol Device:C_Small
- removed C9: CL10A105KB8NNNC, Capacitor_SMD:C_0603_1608Metric, symbol Device:C_Small
- removed U2: VRH1902LTX, Package_TO_SOT_SMD:SOT-23-5, symbol Regulator_Linear:TLV70218_SOT23-5
- added C10, C11, C8, C9: CL10A106KP8NNNC, Capacitor_SMD:C_0603_1608Metric, symbol Device:C
- added D1, D2, D3: BZT52C3V3S, Diode_SMD:D_SOD-323, symbol Device:D_Zener
- added JP1: SolderJumper_2_Open, Jumper:SolderJumper-2_P1.3mm_Bridged_Pad1.0x1.5mm, symbol Jumper:SolderJumper_2_Bridged
- added JP2: SolderJumper_2_Open, Jumper:SolderJumper-2_P1.3mm_Open_Pad1.0x1.5mm, symbol Jumper:SolderJumper_2_Open
- added L1, L2: SDFL2012Q1R0KTF, Inductor_SMD:L_0805_2012Metric, symbol Device:L
- added R3: 0603WAF5603T5E, Resistor_SMD:R_0603_1608Metric, symbol Device:R
- added R4: 0603WAF1303T5E, Resistor_SMD:R_0603_1608Metric, symbol Device:R
- added R5: 0603WAF2403T5E, Resistor_SMD:R_0603_1608Metric, symbol Device:R
- added R6: 0603WAF1103T5E, Resistor_SMD:R_0603_1608Metric, symbol Device:R
- added U3, U4: SK6615C, Package_TO_SOT_SMD:SOT-23-5, symbol neg_symbols:SK6615CS5
Connections:
- net 1V9: now also C11.1, L2.2, R5.1
- net 3V3: now also C9.1, L1.2, R3.1; no longer J1.4 (Pin_4)
- net GND: now also C10.2, C11.2, C8.2, C9.2, D1.2 (A), D2.2 (A), D3.2 (A), JP2.2 (B), R4.2, R6.2, U3.2 (GND), U4.2 (GND)
- net MOSI: now also D3.1 (K)
- net MOTION: now also JP1.2 (B); no longer J1.5 (Pin_5)
- net NCS: now also D2.1 (K)
- net SCLK: now also D1.1 (K)
- new net: L2.1, U4.3 (SW)
- new net: R3.2, R4.1, U3.5 (FB)
- new net: J1.5 (Pin_5), JP1.1 (A), JP2.1 (A)
- new net: R5.2, R6.1, U4.5 (FB)
- new net: L1.1, U3.3 (SW)
- new net VCC: C10.1, C8.1, J1.4 (Pin_4), U3.1 (EN), U3.4 (VIN), U4.1 (EN), U4.4 (VIN)

Commit message: ball v0.1
Parts:
- C6: value CL10A106MA8NRNC -> CL10A106KP8NNNC; LCSC C96446 -> C19702
Changed lines of the file:
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@@
-		)
-	)
-	(global_label "GND"
-		(shape output)
-		(at 135.89 99.06 270)
-		(fields_autoplaced yes)
-		(effects
-			(font
-				(size 1.016 1.016)
-			)
-			(justify right)
-		)
-		(property "Intersheetrefs" "${INTERSHEET_REFS}"
-			(at 135.89 104.5443 90)
-			(effects
-				(font
-					(size 1.27 1.27)
-				)
-				(justify right)
-				(hide yes)
-			)
 		)
 	)
@@
 		)
 	)
-	(global_label "GND"
-		(shape input)
-		(at 111.76 54.61 270)
-		(fields_autoplaced yes)
-		(effects
-			(font
-				(size 1.016 1.016)
-			)
-			(justify right)
-		)
-		(property "Intersheetrefs" "${INTERSHEET_REFS}"
-			(at 111.76 60.0943 90)
-			(effects
-				(font
-					(size 1.27 1.27)
-				)
-				(justify right)
-				(hide yes)
-			)
-		)
-	)
 	(global_label "MISO"
 		(shape output)
@@
 			)
 		)
-		(property "Value" "CL10A106MA8NRNC"
+		(property "Value" "CL10A106KP8NNNC"
 			(at 173.736 71.882 0)
 			(effects
@@
 			)
 		)
-		(property "Datasheet" "https://jlcpcb.com/partdetail/97651-CL10A106MA8NRNC/C96446"
+		(property "Datasheet" "https://jlcpcb.com/partdetail/20411-CL10A106KP8NNNC/C19702"
 			(at 170.18 69.85 0)
 			(effects
@@
 			)
 		)
-		(property "Description" "0603 100u"
+		(property "Description" "0603 10u"
 			(at 184.404 68.834 0)
 			(effects
@@
 			)
 		)
-		(property "LCSC" "C96446"
+		(property "LCSC" "C19702"
 			(at 174.244 68.58 0)
 			(effects
@@
 	(symbol
 		(lib_id "power:GND")
+		(at 111.76 54.61 0)
+		(unit 1)
+		(exclude_from_sim no)
+		(in_bom yes)
+		(on_board yes)
+		(dnp no)
+		(fields_autoplaced yes)
+		(property "Reference" "#PWR010"
+			(at 111.76 60.96 0)
+			(effects
+				(font
+					(size 1.27 1.27)
+				)
+				(hide yes)
+			)
+		)
+		(property "Value" "GND"
+			(at 111.76 59.69 0)
+			(effects
+				(font
+					(size 1.27 1.27)
+				)
+			)
+		)
+		(property "Footprint" ""
+			(at 111.76 54.61 0)
+			(effects
+				(font
+					(size 1.27 1.27)
+				)
+				(hide yes)
+			)
+		)
+		(property "Datasheet" ""
+			(at 111.76 54.61 0)
+			(effects
+				(font
+					(size 1.27 1.27)
+				)
+				(hide yes)
+			)
+		)
+		(property "Description" "Power symbol creates a global label with name \"GND\" , ground"
+			(at 111.76 54.61 0)
+			(effects
+				(font
+					(size 1.27 1.27)
+				)
+				(hide yes)
+			)
+		)
+		(pin "1"
+		)
+		(instances
+			(project "ball_breakout"
+				(path "/f92a57e7-90e7-4a51-b519-f6846ac9b9dd"
+					(reference "#PWR010")
+					(unit 1)
+				)
+			)
+		)
+	)
+	(symbol
+		(lib_id "power:GND")
 		(at 138.43 116.84 0)
 		(unit 1)
@@
 					(unit 1)
 				)
+			)
+		)
+	)
+	(symbol
+		(lib_id "power:GND")
+		(at 135.89 99.06 0)
+		(unit 1)
+		(exclude_from_sim no)
+		(in_bom yes)
+		(on_board yes)
+		(dnp no)
+		(fields_autoplaced yes)
+		(property "Reference" "#PWR09"
+			(at 135.89 105.41 0)
+			(effects
+				(font
+					(size 1.27 1.27)
+				)
+				(hide yes)
+			)
+		)
+		(property "Value" "GND"
+			(at 135.89 104.14 0)
+			(effects
+				(font
+					(size 1.27 1.27)
+				)
+			)
+		)
+		(property "Footprint" ""
+			(at 135.89 99.06 0)
+			(effects
+				(font
+					(size 1.27 1.27)
+				)
+				(hide yes)
+			)
+		)
+		(property "Datasheet" ""
+			(at 135.89 99.06 0)
+			(effects
+				(font
+					(size 1.27 1.27)
+				)
+				(hide yes)
+			)
+		)
+		(property "Description" "Power symbol creates a global label with name \"GND\" , ground"
+			(at 135.89 99.06 0)
+			(effects
+				(font
+					(size 1.27 1.27)
+				)
+				(hide yes)
+			)
+		)
+		(pin "1"
+		)
+		(instances
+			(project "ball_breakout"
+				(path "/f92a57e7-90e7-4a51-b519-f6846ac9b9dd"
+					(reference "#PWR09")
+					(unit 1)
+				)
