File: negL/ball_breakout/ball_breakout.kicad_pcb (KiCad board)
At the start: 2 copper layers, 22 x 25 mm, 14 parts, among them J1 XA-3-2-7P Contact, U1 PAW3395, U2 VRH1902LTX

Commit message: update
Parts:
- removed U2: VRH1902LTX, Package_TO_SOT_SMD:SOT-23-5
- added C10: CL10A106KP8NNNC, Capacitor_SMD:C_0603_1608Metric, B.Cu at (92.2, 92.4)
- added C11: CL10A106KP8NNNC, Capacitor_SMD:C_0603_1608Metric, B.Cu at (88.4, 86.6)
- added D1: BZT52C3V3S, Diode_SMD:D_SOD-323, B.Cu at (103.0, 82.0)
- added D2: BZT52C3V3S, Diode_SMD:D_SOD-323, B.Cu at (103.0, 75.3)
- added D3: BZT52C3V3S, Diode_SMD:D_SOD-323, B.Cu at (103.0, 79.6)
- added JP1: SolderJumper_2_Open, Jumper:SolderJumper-2_P1.3mm_Bridged_Pad1.0x1.5mm, F.Cu at (93.1, 87.2)
- added JP2: SolderJumper_2_Open, Jumper:SolderJumper-2_P1.3mm_Open_Pad1.0x1.5mm, F.Cu at (87.6, 87.0)
- added L1: SDFL2012Q1R0KTF, Inductor_SMD:L_0805_2012Metric, B.Cu at (101.0, 91.8)
- added L2: SDFL2012Q1R0KTF, Inductor_SMD:L_0805_2012Metric, B.Cu at (85.5, 92.0)
- added R3: 0603WAF5603T5E, Resistor_SMD:R_0603_1608Metric, B.Cu at (101.0, 93.6)
- added R4: 0603WAF1303T5E, Resistor_SMD:R_0603_1608Metric, B.Cu at (104.0, 92.8)
- added R5: 0603WAF2403T5E, Resistor_SMD:R_0603_1608Metric, B.Cu at (85.7, 93.7)
- added R6: 0603WAF1103T5E, Resistor_SMD:R_0603_1608Metric, B.Cu at (85.2, 86.5)
- added U3: SK6615C, Package_TO_SOT_SMD:SOT-23-5, B.Cu at (97.1, 92.7)
- added U4: SK6615C, Package_TO_SOT_SMD:SOT-23-5, B.Cu at (89.3, 92.6)
- C8: value CC0603KRX7R9BB104 -> CL10A106KP8NNNC
- C9: value CL10A105KB8NNNC -> CL10A106KP8NNNC
- moved C3 12.4 mm to (86.4, 80.4), turned to 180 degrees
- moved C4 11.0 mm to (86.4, 82.8), turned to 180 degrees
- moved C8 6.79 mm to (93.8, 92.4), turned to 90 degrees
- moved C9 5.70 mm to (101.4, 87.6)
- moved R2 3.57 mm to (103.0, 77.2)
- moved C2 3.53 mm to (86.5, 77.3)
- moved C1 3.37 mm to (86.4, 75.6)
- moved C6 1.60 mm to (86.4, 73.2)
- moved R1 1.04 mm to (102.8, 72.6)
- moved C5 0.91 mm to (86.4, 71.5)
- moved C7 0.77 mm to (104.5, 86.8), turned to -90 degrees
Connections:
- C8 pad 1: GND -> VCC
- C8 pad 2: 3V3 -> GND
- C9 pad 1: 1V9 -> 3V3
- J1 pad 4: 3V3 -> VCC
- J1 pad 5: MOTION -> Net-(J1-Pin_5)
Routing:
- net VCC: track 0.00 -> 16.8 mm, vias 0 -> 1
- net GND: track 63.9 -> 79.6 mm, vias 0 -> 1
- net Net-(U4-FB): track 0.00 -> 12.5 mm
- net 3V3: track 60.4 -> 51.2 mm, vias 4 -> 5
- net Net-(J1-Pin_5): track 0.00 -> 8.57 mm
- net Net-(U3-FB): track 0.00 -> 6.55 mm
- net Net-(U3-SW): track 0.00 -> 4.59 mm
- net 1V9: track 63.0 -> 67.4 mm, vias 2 -> 4
- net MOSI: track 18.0 -> 21.6 mm, vias 1 -> 0
- net MOTION: track 10.8 -> 7.62 mm
- net SCLK: track 8.11 -> 11.2 mm, vias 0 -> 1
- net NCS: track 13.9 -> 16.9 mm, vias 1 -> 0
- net Net-(U4-SW): track 0.00 -> 1.78 mm
- net MISO: track 25.1 -> 26.2 mm, vias 1 -> 3
Other:
- board text removed: "3V3"
- board text removed: "GND"
- board text removed: "MISO"
- board text removed: "MOSI"
- board text removed: "MT"
- board text removed: "NCS"
- board text removed: "SCLK"

Commit message: update
Parts:
- moved C1 1.07 mm to (85.4, 75.7)
- moved C3 1.07 mm to (85.4, 80.4)
- moved C6 1.07 mm to (85.4, 73.3)
- moved C4 1.07 mm to (85.4, 82.8)
- moved C5 1.07 mm to (85.4, 71.6)
- moved C2 1.07 mm to (85.4, 77.3)
Routing:
- net GND: track 79.6 -> 84.7 mm
- net 1V9: track 67.4 -> 70.0 mm
- net VCC: track 16.8 -> 18.4 mm
- net Net-(U1-VDDREG): track 3.91 -> 5.13 mm
Other:
- board text added: "GND"
- board text added: "MISO"
- board text added: "MOSI"
- board text added: "MT"
- board text added: "NCS"
- board text added: "SCLK"
- board text added: "VCC"

Commit message: ball v0.1
Parts:
- C6: value CL10A106MA8NRNC -> CL10A106KP8NNNC
Other:
- board text added: "neg_ball"
- board text added: "v0.1"
Changed lines of the file:
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@@
 		(tags "SOD-323")
 		(property "Reference" "D3"
-			(at 2.095786 0.160674 270)
+			(at 2.095786 0.160674 -90)
 			(layer "B.SilkS")
 			(effects
@@
 		(tags "resistor")
 		(property "Reference" "R2"
-			(at -2.077959 -0.046137 270)
+			(at -2.077959 -0.046137 -90)
 			(layer "B.SilkS")
 			(effects
@@
 		(tags "SOD-323")
 		(property "Reference" "D2"
-			(at 2.114073 0.079782 270)
+			(at 2.114073 0.079782 -90)
 			(layer "B.SilkS")
 			(effects
@@
 			)
 		)
-		(property "Value" "CL10A106MA8NRNC"
+		(property "Value" "CL10A106KP8NNNC"
 			(at 0 -1.43 0)
 			(layer "B.Fab")
@@
 			)
 		)
-		(property "Datasheet" "https://jlcpcb.com/partdetail/97651-CL10A106MA8NRNC/C96446"
+		(property "Datasheet" "https://jlcpcb.com/partdetail/20411-CL10A106KP8NNNC/C19702"
 			(at 0 0 0)
 			(unlocked yes)
@@
 			)
 		)
-		(property "Description" "0603 100u"
+		(property "Description" "0603 10u"
 			(at 0 0 0)
 			(unlocked yes)
@@
 			)
 		)
-		(property "LCSC" "C96446"
+		(property "LCSC" "C19702"
 			(at 0 0 0)
 			(unlocked yes)
@@
 		(effects
 			(font
+				(size 0.6 0.6)
+				(thickness 0.1)
+				(bold yes)
+			)
+			(justify left bottom)
+		)
+	)
+	(gr_text "neg_ball"
+		(at 91.496853 93.914714 0)
+		(layer "F.SilkS")
+		(effects
+			(font
+				(size 1 1)
+				(thickness 0.2)
+				(bold yes)
+			)
+			(justify left bottom)
+		)
+	)
+	(gr_text "v0.1"
+		(at 98.21875 93.799153 0)
+		(layer "F.SilkS" knockout)
+		(effects
+			(font

Commit message: update
Parts:
- moved C7 2.39 mm to (102.5, 85.5), turned to 180 degrees
Routing:
- net 1V9: track 70.0 -> 70.8 mm
Changed lines of the file:
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@@
 	(footprint "Capacitor_SMD:C_0805_2012Metric"
 		(layer "B.Cu")
-		(at 104.490752 86.815177 -90)
+		(at 102.496172 85.500432 180)
 		(descr "Capacitor SMD 0805 (2012 Metric), square (rectangular) end terminal, IPC_7351 nominal, (Body size source: IPC-SM-782 page 76, https://www.pcb-3d.com/wordpress/wp-content/uploads/ipc-sm-782a_amendment_1_and_2.pdf, https://docs.google.com/spreadsheets/d/1BsfQQcO9C6DZCsRaXUlFlo91Tg2WpOkGARC1WS5S8t0/edit?usp=sharing), generated with kicad-footprint-generator")
 		(tags "capacitor")
 		(property "Reference" "C7"
-			(at -2.151277 0.028749 0)
+			(at -2.151277 0.028749 90)
 			(layer "B.SilkS")
 			(effects
@@
 		)
 		(property "Value" "C2012X5R1A336MTJ00E"
-			(at 0 -1.68 90)
+			(at 0 -1.68 0)
 			(layer "B.Fab")
 			(effects
@@
 		)
 		(property "Footprint" "Capacitor_SMD:C_0805_2012Metric"
-			(at 0 0 90)
+			(at 0 0 0)
 			(unlocked yes)
 			(layer "B.Fab")
@@
 		)
 		(property "Datasheet" "https://jlcpcb.com/partdetail/Tdk-C2012X5R1A336MTJ00E/C342635"
-			(at 0 0 90)
+			(at 0 0 0)
 			(unlocked yes)
 			(layer "B.Fab")
@@
 		)
 		(property "Description" "0805 33u"
-			(at 0 0 90)
+			(at 0 0 0)
 			(unlocked yes)
 			(layer "B.Fab")
@@
 		)
 		(property "LCSC" "C342635"
-			(at 0 0 90)
+			(at 0 0 0)
 			(unlocked yes)
 			(layer "B.Fab")
@@
 		)
 		(fp_line
-			(start -1.7 0.98)
-			(end -1.7 -0.98)
+			(start 1.7 0.98)
+			(end -1.7 0.98)
 			(stroke
 				(width 0.05)
@@
 		)
 		(fp_line
-			(start 1.7 0.98)
-			(end -1.7 0.98)
+			(start 1.7 -0.98)
+			(end 1.7 0.98)
 			(stroke
 				(width 0.05)
@@
 		)
 		(fp_line
-			(start -1.7 -0.98)
-			(end 1.7 -0.98)
+			(start -1.7 0.98)
+			(end -1.7 -0.98)
 			(stroke
 				(width 0.05)
@@
 		)
 		(fp_line
-			(start 1.7 -0.98)
-			(end 1.7 0.98)
+			(start -1.7 -0.98)
+			(end 1.7 -0.98)
 			(stroke
 				(width 0.05)
@@
 		)
 		(fp_line
-			(start -1 0.625)
-			(end -1 -0.625)
+			(start 1 0.625)
+			(end -1 0.625)
 			(stroke
 				(width 0.1)
@@
 		)
 		(fp_line
-			(start 1 0.625)
-			(end -1 0.625)
+			(start 1 -0.625)
+			(end 1 0.625)
 			(stroke
 				(width 0.1)
@@
 		)
 		(fp_line
-			(start -1 -0.625)
-			(end 1 -0.625)
+			(start -1 0.625)
+			(end -1 -0.625)
 			(stroke
 				(width 0.1)
@@
 		)
 		(fp_line
-			(start 1 -0.625)
-			(end 1 0.625)
+			(start -1 -0.625)
+			(end 1 -0.625)
 			(stroke
 				(width 0.1)
@@
 		)
 		(fp_text user "${REFERENCE}"
-			(at 0 0 90)
+			(at 0 0 0)
 			(layer "B.Fab")
 			(effects
@@
 		)
 		(pad "1" smd roundrect
-			(at -0.95 0 270)
+			(at -0.95 0 180)
 			(size 1 1.45)
 			(layers "B.Cu" "B.Paste" "B.Mask")
@@
 		)
 		(pad "2" smd roundrect
-			(at 0.95 0 270)
+			(at 0.95 0 180)
 			(size 1 1.45)
 			(layers "B.Cu" "B.Paste" "B.Mask")
@@
 	)
 	(segment
+		(start 105.20625 83.740354)
+		(end 105.20625 83.16375)
+		(width 0.4)
+		(layer "B.Cu")
+		(net 1)
+	)
+	(segment
 		(start 84.434412 93.254124)
 		(end 84.891864 93.711576)
@@
 	)
 	(segment
-		(start 84.485458 91.955819)
-		(end 84.434412 92.006865)
+		(start 105.20625 83.16375)
+		(end 105.20625 74.199101)
 		(width 0.4)
 		(layer "B.Cu")
@@
 	)
 	(segment
-		(start 104.490752 85.865177)
-		(end 105.20625 85.149679)
+		(start 84.485458 91.955819)
+		(end 84.434412 92.006865)
 		(width 0.4)
 		(layer "B.Cu")
@@
 	)
 	(segment
-		(start 85.634746 93.794409)
-		(end 85.551913 93.711576)
-		(width 0.4)
-		(layer "B.Cu")
-		(net 1)
-	)
-	(segment
-		(start 105.20625 74.199101)
-		(end 103.625228 72.618079)
+		(start 103.446172 85.623634)
+		(end 104.587715 86.765177)
 		(width 0.4)
 		(layer "B.Cu")
@@
 	)
 	(segment
-		(start 105.20625 85.149679)
-		(end 105.20625 74.199101)
+		(start 85.634746 93.794409)
+		(end 85.551913 93.711576)
 		(width 0.4)
 		(layer "B.Cu")
@@
 	)
 	(segment
-		(start 104.587715 85.96214)
-		(end 104.490752 85.865177)
+		(start 105.20625 74.199101)
+		(end 103.625228 72.618079)
 		(width 0.4)
 		(layer "B.Cu")
@@
 	)
 	(segment
-		(start 104.587715 86.765177)
-		(end 104.587715 85.96214)
+		(start 103.446172 85.500432)
+		(end 105.20625 83.740354)
+		(width 0.4)
+		(layer "B.Cu")
+		(net 1)
+	)
+	(segment
+		(start 103.446172 85.500432)
+		(end 103.446172 85.623634)
 		(width 0.4)
 		(layer "B.Cu")
@@
 	)
 	(segment
-		(start 86.65599 84.354375)
-		(end 86.049871 84.960494)
+		(start 100.6 86.446604)
+		(end 100.6 87.496596)
 		(width 0.4)
 		(layer "B.Cu")
@@
 	)
 	(segment
-		(start 86.049871 84.354375)
+		(start 86.65599 84.354375)
 		(end 86.049871 84.960494)
 		(width 0.4)
@@
 	)
 	(segment
-		(start 103.099686 84.100262)
-		(end 103.099686 84.971893)
-		(width 0.4)
-		(layer "B.Cu")
-		(net 14)
-	)
-	(segment
-		(start 104.0308 81.973125)
-		(end 104.0308 83.169148)
+		(start 86.049871 84.354375)
+		(end 86.049871 84.960494)
 		(width 0.4)
 		(layer "B.Cu")
@@
 	)
 	(segment
-		(start 103.099686 84.971893)
-		(end 103.099686 85.401428)
-		(width 0.4)
-		(layer "B.Cu")
-		(net 14)
-	)
-	(segment
 		(start 97.1919 89.8075)
 		(end 99.441503 87.557897)
@@
 	)
 	(segment
-		(start 102.81777 85.661881)
-		(end 103.099686 85.943797)
+		(start 101.546172 85.500432)
+		(end 101.634518 85.500432)
 		(width 0.4)
 		(layer "B.Cu")
@@
 	)
 	(segment
+		(start 104.0308 83.10415)
+		(end 104.0308 81.973125)
+		(width 0.4)
+		(layer "B.Cu")
+		(net 14)
+	)
+	(segment
 		(start 104.60625 75.934081)
 		(end 104.012963 75.340794)
@@
 	)
 	(segment
-		(start 100.661301 87.557897)
-		(end 102.81777 85.401428)
+		(start 100.6 87.496596)
+		(end 100.661301 87.557897)
 		(width 0.4)
 		(layer "B.Cu")
@@
 	)
 	(segment
-		(start 103.099686 86.374111)
+		(start 101.546172 85.500432)
+		(end 102.809815 86.764075)
+		(width 0.4)
+		(layer "B.Cu")
+		(net 14)
+	)
+	(segment
+		(start 103.48965 86.764075)
 		(end 104.490752 87.765177)
 		(width 0.4)
@@
 	)
 	(segment
+		(start 101.546172 85.500432)
+		(end 100.6 86.446604)
+		(width 0.4)
+		(layer "B.Cu")
+		(net 14)
+	)
+	(segment
 		(start 86.049871 84.960494)
 		(end 86.049871 86.535711)
@@
 	)
 	(segment
-		(start 102.81777 85.401428)
-		(end 103.099686 85.401428)
-		(width 0.4)
-		(layer "B.Cu")
-		(net 14)
-	)
-	(segment
 		(start 86.049871 86.535711)
 		(end 86.049172 86.53641)
@@
 	)
 	(segment
-		(start 103.099686 85.401428)
-		(end 103.099686 85.943797)
-		(width 0.4)
-		(layer "B.Cu")
-		(net 14)
-	)
-	(segment
 		(start 86.290903 90.985268)
 		(end 88.954528 90.985268)
@@
 	)
 	(segment
-		(start 102.81777 85.253809)
-		(end 103.099686 84.971893)
-		(width 0.4)
-		(layer "B.Cu")
-		(net 14)
-	)
-	(segment
 		(start 87.346598 84.354375)
 		(end 86.049871 84.354375)
@@
 	)
 	(segment
-		(start 102.81777 85.401428)
-		(end 102.81777 85.253809)
-		(width 0.4)
-		(layer "B.Cu")
-		(net 14)
-	)
-	(segment
-		(start 102.81777 85.401428)
-		(end 102.81777 85.661881)
-		(width 0.4)
-		(layer "B.Cu")
-		(net 14)
-	)
-	(segment
 		(start 94.402357 91.061904)
 		(end 95.937496 91.061904)
@@
 	)
 	(segment
-		(start 104.0308 83.169148)
-		(end 103.099686 84.100262)
-		(width 0.4)
-		(layer "B.Cu")
-		(net 14)
-	)
-	(segment
 		(start 104.60625 79.016875)
 		(end 104.60625 75.934081)
@@
 	)
 	(segment
+		(start 102.809815 86.764075)
+		(end 103.48965 86.764075)
+		(width 0.4)
+		(layer "B.Cu")
+		(net 14)
+	)
+	(segment
 		(start 85.8819 86.703682)
 		(end 86.049172 86.53641)
@@
 	)
 	(segment
-		(start 103.099686 85.943797)
-		(end 103.099686 86.374111)
+		(start 101.634518 85.500432)
+		(end 104.0308 83.10415)
 		(width 0.4)
 		(layer "B.Cu")

Commit message: update
Parts:
- removed C8, C9: CL10A106KP8NNNC, Capacitor_SMD:C_0603_1608Metric
- removed D1, D2, D3: BZT52C3V3S, Diode_SMD:D_SOD-323
- removed L1: SDFL2012Q1R0KTF, Inductor_SMD:L_0805_2012Metric
- removed R3: 0603WAF5603T5E, Resistor_SMD:R_0603_1608Metric
- removed R4: 0603WAF1303T5E, Resistor_SMD:R_0603_1608Metric
- removed U3: SK6615C, Package_TO_SOT_SMD:SOT-23-5
- moved JP2 19.7 mm to (103.2, 75.1)
- moved JP1 13.9 mm to (103.2, 77.6), turned to 180 degrees
- moved C7 7.49 mm to (101.2, 92.9)
- moved C10 4.41 mm to (96.6, 92.9)
- moved U4 3.69 mm to (93.0, 92.8)
- moved R2 3.48 mm to (103.2, 80.7)
Connections:
- C10 pad 1: VCC -> 3V3
- J1 pad 4: VCC -> 3V3
- U4 pad 1: VCC -> 3V3
- U4 pad 4: VCC -> 3V3
Routing:
- net GND: track 84.4 -> 20.9 mm, vias 1 -> 0
- net 1V9: track 70.8 -> 22.2 mm, vias 4 -> 0
- net Net-(J1-Pin_5): track 8.57 -> 31.7 mm
- net VCC: track 18.4 -> 0.00 mm, vias 1 -> 0
- net 3V3: track 51.2 -> 36.1 mm, vias 5 -> 2
- net Net-(U3-FB): track 6.55 -> 0.00 mm
- net MOSI: track 21.5 -> 27.5 mm
- net MISO: track 26.2 -> 32.1 mm, vias 3 -> 0
- net Net-(U1-VDDREG): track 5.13 -> 0.00 mm
- net Net-(U3-SW): track 4.59 -> 0.00 mm
- net Net-(U4-FB): track 12.5 -> 8.20 mm
- net NCS: track 16.9 -> 14.9 mm, vias 0 -> 1
- net Net-(U4-SW): track 1.78 -> 0.00 mm
- net MOTION: track 7.62 -> 8.73 mm, vias 0 -> 1
- net SCLK: track 10.9 -> 9.79 mm, vias 1 -> 0
