File: negL/pcb_R/pcb_R.kicad_sch (KiCad schematic)
At the start: 112 parts, among them J1 MJ-4PP-9, J2 FH-1x4SG/RH, J3 XA-3-2-7P, Q1 AO3401A, Q2 AO3400A, SW1 TVBP06-B043CB-B, SW2 EVQWGD001, SW3 SS-12D00G3, SW4 SS-12D00G3, U1 nice_nano, U2 74HC595, U3 AE-XCL103-3V3

Commit message: update
Parts:
- removed JP2: LED Jumper, Jumper:SolderJumper-2_P1.3mm_Bridged_Pad1.0x1.5mm, symbol Jumper:SolderJumper_2_Bridged
- removed JP4: ~, Jumper:SolderJumper-2_P1.3mm_Open_Pad1.0x1.5mm, symbol Jumper:SolderJumper_2_Open
- removed Q1: AO3401A, Package_TO_SOT_SMD:SOT-23, symbol Transistor_FET:AO3401A
- removed Q2: AO3400A, Package_TO_SOT_SMD:SOT-23, symbol Transistor_FET:AO3400A
- removed U3: AE-XCL103-3V3, neg_footprints:AE-XCL103-3V3_Vertical, symbol neg_symbols:AE-XCL103-3V3
- added BT2: JST_PH_S2B, Connector_JST:JST_PH_S2B-PH-K_1x02_P2.00mm_Horizontal, symbol Device:Battery_Cell
- added C1, C2, C3: CL10A106KP8NNNC, Capacitor_SMD:C_0603_1608Metric, symbol Device:C
- added C4: CL10A226MQ8NRNC, Capacitor_SMD:C_0603_1608Metric, symbol Device:C
- added D31: SS12, Diode_SMD:D_SMA, symbol Device:D
- added IC1: SN74LVC4245A, neg_footprints:TSSOP-24, symbol neg_symbols:SN74LVC4245A
- added JP1, JP12, JP13, JP2: ~, Jumper:SolderJumper-2_P1.3mm_Open_Pad1.0x1.5mm, symbol Jumper:SolderJumper_2_Open
- added JP10: LED switch input, Jumper:SolderJumper-2_P1.3mm_Open_Pad1.0x1.5mm, symbol Jumper:SolderJumper_2_Open
- added JP11: LED_VCC Direct, Jumper:SolderJumper-2_P1.3mm_Open_Pad1.0x1.5mm, symbol Jumper:SolderJumper_2_Open
- added JP9: LED_VCC 5V, Jumper:SolderJumper-2_P1.3mm_Open_Pad1.0x1.5mm, symbol Jumper:SolderJumper_2_Open
- added L1, L2: SDFL1608Q4R7KTF, Inductor_SMD:L_0603_1608Metric, symbol Device:L
- added Q1: AO3400A, Package_TO_SOT_SMD:SOT-23, symbol Transistor_FET:AO3400A
- added R4: 0603WAF4992T5E, Resistor_SMD:R_0603_1608Metric, symbol Device:R
- added R5: 0603WAF5601T5E, Resistor_SMD:R_0603_1608Metric, symbol Device:R
- added R6: 0603WAF1003T5E, Resistor_SMD:R_0603_1608Metric, symbol Device:R
- added R7: 0603WAF1802T5E, Resistor_SMD:R_0603_1608Metric, symbol Device:R
- added U3, U4: TLV61070ADBV, Package_TO_SOT_SMD:SOT-23-6, symbol Regulator_Switching:TLV61070ADBV
- J3, SW2, SW3, SW4: now left out of the parts list
- renumbered JP1 to JP4
Connections:
- net BALL_MOTION: now also U1.25 (P1.01-LF); no longer U1.17 (P0.31-LF)
- net BAT+: now also SW3.1 (A), BT2.1 (+), D31.2 (A), JP1.1 (A)
- net BAT-: now also Q1.3 (D)
- net GND: now also C1.2, C2.2, IC1.11 (GND), IC1.12 (GND), IC1.13 (GND), R5.2, U3.2 (GND)
- net LED: now also JP12.1 (A), JP13.1 (A); no longer LED1.3 (DIN)
- net LED_POWER: now also U1.17 (P0.31-LF), JP10.2 (B); no longer R3.1, SW4.3 (C), U1.25 (P1.01-LF)
- net VCC: now also SW4.1 (A), IC1.1 (VCCA), JP9.1 (A)
- net LED_VCC: now reaches LED1.1 (VDD), LED10.1 (VDD), LED11.1 (VDD), LED12.1 (VDD), LED13.1 (VDD), LED14.1 (VDD), LED15.1 (VDD), LED16.1 (VDD), LED17.1 (VDD), LED18.1 (VDD), LED19.1 (VDD), LED2.1 (VDD), LED20.1 (VDD), LED21.1 (VDD), LED22.1 (VDD), LED23.1 (VDD), LED24.1 (VDD), LED25.1 (VDD), LED26.1 (VDD), LED27.1 (VDD), LED28.1 (VDD), LED29.1 (VDD), LED3.1 (VDD), LED4.1 (VDD), LED5.1 (VDD), LED6.1 (VDD), LED7.1 (VDD), LED8.1 (VDD), LED9.1 (VDD)
- net LED_VCC: now also C2.1, IC1.23 (VCCB), IC1.24 (VCCB), JP11.2 (B), R4.1, U3.5 (V_{OUT})
- net at SW4.2 (B): now also JP11.1 (A), U3.3 (EN)
- net at SW3.2 (B): now also Q1.1 (G)
- net at BT1.2 (-), SW3.3 (C): now also BT2.2 (-), C3.2, C4.2, Q1.2 (S), R7.2, U4.2 (GND)
- new net: L2.2, U4.1 (SW)
- new net: C3.1, JP2.1 (A), L2.1, U4.3 (EN), U4.6 (V_{IN})
- new net: R6.2, R7.1, U4.4 (V_{FB})
- new net: C4.1, D31.1 (K), JP3.1 (A), R6.1, U4.5 (V_{OUT})
- new net: JP10.1 (A), R3.1, SW4.3 (C)
- new net: L1.2, U3.1 (SW)
- new net: R4.2, R5.1, U3.4 (V_{FB})
- new net: C1.1, JP9.2 (B), L1.1, U3.6 (V_{IN})
- new net: BT1.1 (+), JP1.2 (B), JP2.2 (B)
- new net: IC1.3 (A1), JP13.2 (B)
- new net: IC1.21 (B1), JP12.2 (B), LED1.3 (DIN)
- no-connect marks 5 -> 21
Other:
- note added: "Jumper config [Power] JP1: enables direct output from battery. Use this for 14500 battery. JP2: enables boost converter to 3.3v. Use this for AA battery. JP3: Debug purpose. Shorts diode to block charging AA battery. NOTE: JP1 and JP2 are exclusive! [Matrix] JP4: Jumper to detect hand. Enables COL0, ROW3. [TRRS] JP5-8: Exists for ProMicro RP2040, whose uart pin cannot be selected. Usually, jump J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"
- note removed: "JP3: Enables direct output from battery. Intented to use with 14500 battery. JP4: Enables step up converter to 3.3V. Intended to use with normal AA battery."
- note removed: "NOTE: XCL103's max current is 0.25A at 1.5V, which is not enough to light all LEDs in max brightness"
- note removed: "Short JP7 and JP8 for right hand"
- moved on the sheet: J1, J2, J3, JP5, JP6, JP7, JP8, LED1, LED10, LED11, LED12, LED13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

Commit message: update
Parts:
- D1, D10, D11, D12, D13, D14, D15, D16, D17, D18, D19, D2, D20, D21, D22, D23, D24, D25, D26, D27, D28, D29, D3, D30, D4, D5, D6, D7, D8, D9: LCSC C81598 -> C7420318
- D31: value SS12 -> SS14; LCSC C18199177 -> C2480
Connections:
- net BAT+: now also D31.1 (K); no longer BT2.1 (+), D31.2 (A), JP1.1 (A), SW3.1 (A)
- net at C4.1, JP3.1 (A), R6.1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: now also BT2.1 (+), D31.2 (A), JP1.1 (A), SW3.1 (A); no longer D31.1 (K)
Other:
- note added: "Jumper config [Power] JP1: enables direct output from battery. Use this for 14500 battery. JP2: enables boost converter to 3.3v. Use this for AA battery. JP3: Shorts the diode that allows current to flow only in the discharging direction. Only jump when using LiPo or Li-ion batteries. NOTE: JP1 and JP2 are exclusive! [Matrix] JP4: Jumper to detect hand. Enables COL0, ROW3. [TRRS] JP5-8: Exists fo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"
- note removed: "Jumper config [Power] JP1: enables direct output from battery. Use this for 14500 battery. JP2: enables boost converter to 3.3v. Use this for AA battery. JP3: Debug purpose. Shorts diode to block charging AA battery. NOTE: JP1 and JP2 are exclusive! [Matrix] JP4: Jumper to detect hand. Enables COL0, ROW3. [TRRS] JP5-8: Exists for ProMicro RP2040, whose uart pin cannot be selected. Usually, jump J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"
