File: negL/pcb_R/pcb_R.kicad_sch (KiCad schematic)
At the start: 130 parts, among them IC1 SN74LVC4245A, J1 MJ-4PP-9, J2 FH-1x4SG/RH, J3 XA-3-2-7P, Q1 AO3400A, SW1 TVBP06-B043CB-B, SW2 EVQWGD001, SW3 SS-12D00G3, SW4 SS-12D00G3, U1 nice_nano, U2 74HC595, U3 TLV61070ADBV, U4 TLV61070ADBV

Commit message: update
Parts:
- added D32: 1N4148W, Diode_SMD:D_SOD-123, symbol Diode:1N4148W
Connections:
- net ROW3: now also D32.1 (K); no longer JP4.2 (B)
- new net: D32.2 (A), JP4.2 (B)
Other:
- note removed: "Jumper config [Power] JP1: enables direct output from battery. Use this for 14500 battery. JP2: enables boost converter to 3.3v. Use this for AA battery. JP3: Shorts the diode that allows current to flow only in the discharging direction. Only jump when using LiPo or Li-ion batteries. NOTE: JP1 and JP2 are exclusive! [Matrix] JP4: Jumper to detect hand. Enables COL0, ROW3. [TRRS] JP5-8: Exists fo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"
Changed lines of the file:
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@@
 	(wire
 		(pts
-			(xy 114.3 97.79) (xy 114.3 110.49)
+			(xy 114.3 97.79) (xy 114.3 102.87)
 		)
 		(stroke
@@
 		)
 	)
-	(text "Jumper config\n\n[Power]\nJP1: enables direct output from battery. Use this for 14500 battery.\nJP2: enables boost converter to 3.3v. Use this for AA battery.\nJP3: Shorts the diode that allows current to flow only in the discharging direction. Only jump when using LiPo or Li-ion batteries.\n\nNOTE: JP1 and JP2 are exclusive!\n\n[Matrix]\nJP4: Jumper to detect hand. Enables COL0, ROW3.\n\n[TRRS]\nJP5-8: Exists for ProMicro RP2040, whose uart pin cannot be selected. Usually, jump JP5 and JP6.\n\n[LED]\nJP9,10: Jump these to enable 5V boost converter for LED VCC.\nJP11: Debug purpose. Jump this to disable boost converter and just use vcc of promicro.\n\nNOTE: [JP9 and JP10] and JP11 are exclusive!\n\nJP12: Enables level shifting of LED signal. This should be jumped if LED VCC boost converter is enabled.\nJP13: Disables level shifting of LED signal."
-		(exclude_from_sim no)
-		(at 15.748 314.198 0)
-		(effects
-			(font
-				(size 1.27 1.27)
-				(thickness 0.254)
-				(bold yes)
-			)
-			(justify left)
-		)
-	)
 	(global_label "MISO"
 		(shape input)
@@
 					(unit 1)
 				)
+			)
+		)
+	)
+	(symbol
+		(lib_id "Diode:1N4148W")
+		(at 114.3 106.68 90)
+		(unit 1)
+		(exclude_from_sim no)
+		(in_bom yes)
+		(on_board yes)
+		(dnp no)
+		(property "Reference" "D32"
+			(at 110.998 106.68 0)
+			(effects
+				(font
+					(size 1.27 1.27)
+				)
+			)
+		)
+		(property "Value" "1N4148W"
+			(at 110.49 106.68 0)
+			(effects
+				(font
+					(size 1.27 1.27)
+				)
+				(hide yes)
+			)
+		)
+		(property "Footprint" "Diode_SMD:D_SOD-123"
+			(at 118.745 106.68 0)
+			(effects
+				(font
+					(size 1.27 1.27)
+				)
+				(hide yes)
+			)
+		)
+		(property "Datasheet" "https://www.vishay.com/docs/85748/1n4148w.pdf"
+			(at 114.3 106.68 0)
+			(effects
+				(font
+					(size 1.27 1.27)
+				)
+				(hide yes)
+			)
+		)
+		(property "Description" "75V 0.15A Fast Switching Diode, SOD-123"
+			(at 114.3 106.68 0)
+			(effects
+				(font
+					(size 1.27 1.27)
+				)
+				(hide yes)
+			)
+		)
+		(property "Sim.Device" "D"
+			(at 114.3 106.68 0)
+			(effects
+				(font
+					(size 1.27 1.27)
+				)
+				(hide yes)
+			)
+		)
+		(property "Sim.Pins" "1=K 2=A"
+			(at 114.3 106.68 0)
+			(effects
+				(font
+					(size 1.27 1.27)
+				)
+				(hide yes)
+			)
+		)
+		(property "LCSC" "C7420318"
+			(at 110.998 106.68 0)
+			(effects
+				(font
+					(size 1.27 1.27)
+				)
+				(hide yes)
+			)
+		)
+		(pin "1"
+		)
+		(pin "2"
+		)
+		(instances
+			(project "pcb_R"
+				(path "/9ab7ca09-b2ea-4853-bd3f-96554febaf98"
+					(reference "D32")
+					(unit 1)
+				)

Commit message: update
Parts:
- removed JP10: LED switch input, Jumper:SolderJumper-2_P1.3mm_Open_Pad1.0x1.5mm, symbol Jumper:SolderJumper_2_Open
- removed Q1: AO3400A, Package_TO_SOT_SMD:SOT-23, symbol Transistor_FET:AO3400A
- removed SW2: EVQWGD001, neg_footprints:EVQWGD001_EC12, symbol neg_symbols:EVQWGD001
- added MT1, MT10, MT11, MT2, MT3, MT4, MT5, MT6, MT7, MT8, MT9: MountingHole, neg_footprints:M2_SPACER, symbol Mechanical:MountingHole
- added Q1, Q2, Q3: AO3401A, Package_TO_SOT_SMD:SOT-23, symbol Transistor_FET:AO3401A
- added SW2: EVQWGD001_EC12, neg_footprints:EVQWGD001_EC12, symbol neg_symbols:EVQWGD001_EC12
Connections:
- net BAT-: now also BT1.2 (-), BT2.2 (-), C3.2, C4.2, R7.2, SW3.1 (A), U4.2 (GND)
- net COL0: now also SW2.S1
- net ENC_A: now also SW2.A
- net ENC_B: now also SW2.B
- net LED_POWER: now also R3.1, SW4.3 (C)
- net LED_VCC: now also Q1.3 (D); no longer JP11.2 (B)
- net VCC: now also JP11.1 (A), SW2.C
- net at BT2.1 (+), C4.1, JP1.1 (A)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: now also SW3.3 (C), Q3.3 (D); no longer D31.2 (A), JP3.1 (A), SW3.1 (A)
- net at D30.2 (A): now also SW2.S2
- net at SW4.2 (B), U3.3 (EN): now also Q1.1 (G); no longer JP11.1 (A)
- net at SW3.2 (B): now also Q2.1 (G), Q3.1 (G)
- new net: D31.2 (A), JP3.1 (A), Q2.3 (D)
- new net: Q2.2 (S), Q3.2 (S)
- new net: JP11.2 (B), Q1.2 (S)
Other:
- note added: "Ball"
- note added: "Key Matrix"
- note added: "LED"
- note added: "MCU"
- note added: "Mount"
- note added: "OLED"
- note added: "Power"
- note added: "Reset"
- note added: "TRRS"
- moved on the sheet: BT1, BT2, C3, C4, D31, IC1, J1, J2, J3, JP1, JP12, JP13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

Commit message: update
Parts:
- Q1, Q2, Q3: LCSC (none) -> C15127
- SW2: footprint neg_footprints:EVQWGD001_EC12 -> neg_footprints:choc_encoder
- renumbered D32 to D31, D31 to D32, JP9 to JP10, JP12 to JP11, JP13 to JP12, JP11 to JP9
Changed lines of the file:
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@@
 			)
 		)
-		(property "Footprint" "neg_footprints:EVQWGD001_EC12"
+		(property "Footprint" "neg_footprints:choc_encoder"
 			(at 398.78 142.24 0)
 			(effects
@@
 			)
 		)
+		(property "LCSC" "C15127"
+			(at 162.5601 46.99 0)
+			(effects
+				(font
+					(size 1.27 1.27)
+				)
+				(hide yes)
+			)
+		)
 		(pin "2"
 		)
@@
 			)
 		)
+		(property "LCSC" "C15127"
+			(at 149.8599 46.99 0)
+			(effects
+				(font
+					(size 1.27 1.27)
+				)
+				(hide yes)
+			)
+		)
 		(pin "2"
 		)
@@
 		(on_board yes)
 		(dnp no)
-		(property "Reference" "JP11"
+		(property "Reference" "JP9"
 			(at 285.75 212.0899 90)
 			(effects
@@
 			(project "pcb_R"
 				(path "/9ab7ca09-b2ea-4853-bd3f-96554febaf98"
-					(reference "JP11")
+					(reference "JP9")
 					(unit 1)
 				)
@@
 		(on_board yes)
 		(dnp no)
-		(property "Reference" "JP13"
+		(property "Reference" "JP12"
 			(at 46.228 235.204 0)
 			(effects
@@
 			(project "pcb_R"
 				(path "/9ab7ca09-b2ea-4853-bd3f-96554febaf98"
-					(reference "JP13")
+					(reference "JP12")
 					(unit 1)
 				)
@@
 		(on_board yes)
 		(dnp no)
-		(property "Reference" "D32"
+		(property "Reference" "D31"
 			(at 375.158 102.87 0)
 			(effects
@@
 			(project "pcb_R"
 				(path "/9ab7ca09-b2ea-4853-bd3f-96554febaf98"
-					(reference "D32")
+					(reference "D31")
 					(unit 1)
 				)
@@
 			)
 		)
+		(property "LCSC" "C15127"
+			(at 287.02 262.8901 0)
+			(effects
+				(font
+					(size 1.27 1.27)
+				)
+				(hide yes)
+			)
+		)
 		(pin "2"
 		)
@@
 		(on_board yes)
 		(dnp no)
-		(property "Reference" "JP9"
+		(property "Reference" "JP10"
 			(at 326.39 212.0899 90)
 			(effects
@@
 			(project "pcb_R"
 				(path "/9ab7ca09-b2ea-4853-bd3f-96554febaf98"
-					(reference "JP9")
+					(reference "JP10")
 					(unit 1)
 				)
@@
 		(on_board yes)
 		(dnp no)
-		(property "Reference" "JP12"
+		(property "Reference" "JP11"
 			(at 37.338 235.204 0)
 			(effects
@@
 			(project "pcb_R"
 				(path "/9ab7ca09-b2ea-4853-bd3f-96554febaf98"
-					(reference "JP12")
+					(reference "JP11")
 					(unit 1)
 				)
@@
 		(on_board yes)
 		(dnp no)
-		(property "Reference" "D31"
+		(property "Reference" "D32"
 			(at 133.35 36.83 0)
 			(effects
@@
 			(project "pcb_R"
 				(path "/9ab7ca09-b2ea-4853-bd3f-96554febaf98"
-					(reference "D31")
+					(reference "D32")
 					(unit 1)
 				)

Commit message: update
Changed lines of the file:
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@@
 	(wire
 		(pts
+			(xy 50.8 81.28) (xy 50.8 86.36)
+		)
+		(stroke
+			(width 0)
+			(type default)
+		)
+	)
+	(wire
+		(pts
 			(xy 176.53 107.95) (xy 161.29 107.95)
 		)
@@
 	(global_label "BALL_MOTION"
 		(shape input)
-		(at 50.8 81.28 270)
+		(at 50.8 86.36 270)
 		(fields_autoplaced yes)
 		(effects
@@
 		)
 		(property "Intersheetrefs" "${INTERSHEET_REFS}"
-			(at 50.8 93.5861 90)
+			(at 50.8 98.6661 90)
 			(effects
 				(font

Commit message: update
Parts:
- added MT12: MountingHole, neg_footprints:M2_SPACER, symbol Mechanical:MountingHole
Changed lines of the file:
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@@
 	(rectangle
 		(start 27.94 350.52)
-		(end 152.4 364.49)
+		(end 163.83 364.49)
 		(stroke
 			(width 0)
@@
 					(unit 1)
 				)
+			)
+		)
+	)
+	(symbol
+		(lib_id "Mechanical:MountingHole")
+		(at 153.67 356.87 0)
+		(unit 1)
+		(exclude_from_sim yes)
+		(in_bom no)
+		(on_board yes)
+		(dnp no)
+		(fields_autoplaced yes)
+		(property "Reference" "MT12"
+			(at 156.21 355.5999 0)
+			(effects
+				(font
+					(size 1.27 1.27)
+				)
+				(justify left)
+			)
+		)
+		(property "Value" "MountingHole"
+			(at 156.21 358.1399 0)
+			(effects
+				(font
+					(size 1.27 1.27)
+				)
+				(justify left)
+				(hide yes)
+			)
+		)
+		(property "Footprint" "neg_footprints:M2_SPACER"
+			(at 153.67 356.87 0)
+			(effects
+				(font
+					(size 1.27 1.27)
+				)
+				(hide yes)
+			)
+		)
+		(property "Datasheet" "~"
+			(at 153.67 356.87 0)
+			(effects
+				(font
+					(size 1.27 1.27)
+				)
+				(hide yes)
+			)
+		)
+		(property "Description" "Mounting Hole without connection"
+			(at 153.67 356.87 0)
+			(effects
+				(font
+					(size 1.27 1.27)
+				)
+				(hide yes)
+			)
+		)
+		(instances
+			(project "pcb_R"
+				(path "/9ab7ca09-b2ea-4853-bd3f-96554febaf98"
+					(reference "MT12")
+					(unit 1)
+				)

Commit message: update
Parts:
- added JP15: (no value), Jumper:SolderJumper-2_P1.3mm_Open_Pad1.0x1.5mm, symbol Jumper:SolderJumper_2_Open
- added JP2, JP5: ~, Jumper:SolderJumper-2_P1.3mm_Open_Pad1.0x1.5mm, symbol Jumper:SolderJumper_2_Open
- JP13: renamed from JP9; value LED_VCC Direct -> (none)
- JP14: renamed from JP10; value LED_VCC 5V -> (none)
- JP6: renamed from JP4; value Hand Jumper -> (none)
- renumbered JP3 to JP1, JP8 to JP10, JP1 to JP3, JP2 to JP4, JP5 to JP7, JP6 to JP8, JP7 to JP9
Connections:
- net LED: now also IC1.3 (A1); no longer JP12.1 (A)
- net LED_VCC: now also JP15.2 (B); no longer C2.1, R4.1, U3.5 (V_{OUT})
- net at JP12.2 (B): now also JP11.2 (B), LED1.3 (DIN); no longer IC1.3 (A1)
- new net: C4.1, JP5.1 (A), R6.1, U4.5 (V_{OUT})
- new net: C2.1, JP15.1 (A), R4.1, U3.5 (V_{OUT})
- new net: JP2.1 (A), JP3.1 (A), JP5.2 (B), Q3.3 (D), SW3.3 (C)
- new net: BT2.1 (+), JP2.2 (B)
- new net: IC1.21 (B1), JP12.1 (A)
Other:
- moved on the sheet: BT2, IC1

Commit message: update
Parts:
- added JP13: ~, Jumper:SolderJumper-2_P1.3mm_Open_Pad1.0x1.5mm, symbol Jumper:SolderJumper_2_Open
- JP14: renamed from JP13; value (none) -> ~
- JP15: renamed from JP14; value (none) -> ~
- JP16: renamed from JP15; value (none) -> ~
- JP6: value (none) -> ~
Connections:
- net GND: now also JP13.2 (B)
- net VCC: now also IC1.2 (DIR), JP12.1 (A)
- net at JP11.2 (B), LED1.3 (DIN): now also IC1.21 (B1); no longer JP12.2 (B)
- net at IC1.22 (~{OE}): now also JP12.2 (B), JP13.1 (A)
- no-connect marks 21 -> 19
Other:
- moved on the sheet: IC1, JP11

Commit message: update
Parts:
- removed D32: SS14, Diode_SMD:D_SMA, symbol Device:D
- removed Q1, Q2: AO3401A, Package_TO_SOT_SMD:SOT-23, symbol Transistor_FET:AO3401A
- added C5: CL10C220JB8NNNC, Capacitor_SMD:C_0603_1608Metric, symbol Device:C
- added Q1, Q2: AO3400A, Package_TO_SOT_SMD:SOT-23, symbol Transistor_FET:AO3400A
- added U6: LM66100DCKR, Package_TO_SOT_SMD:SOT-363_SC-70-6, symbol Power_Management:LM66100DCK
- C1: value CL10A106KP8NNNC -> C1608X5R1A225K080AC; LCSC C19702 -> (none)
- C2: value CL10A106KP8NNNC -> C3216X5R1A226M160AC; footprint Capacitor_SMD:C_0603_1608Metric -> Capacitor_SMD:C_1206_3216Metric; LCSC C19702 -> (none)
- C3: value CL10A106KP8NNNC -> GRM155R60J106ME11D; footprint Capacitor_SMD:C_0603_1608Metric -> Capacitor_SMD:C_0402_1005Metric
- C4: value CL10A226MQ8NRNC -> GRM32ER61A107ME20L; footprint Capacitor_SMD:C_0603_1608Metric -> Capacitor_SMD:C_1210_3225Metric
- IC1: value SN74LVC4245A -> SN74LVC4245APWR; footprint neg_footprints:TSSOP-24 -> Package_SO:TSSOP-24_4.4x7.8mm_P0.65mm; LCSC C7859 -> (none)
- L1: value SDFL1608Q4R7KTF -> XFL4020-102MEB; footprint Inductor_SMD:L_0603_1608Metric -> Inductor_SMD:L_Coilcraft_XxL4020; LCSC C1034 -> (none)
- L2: value SDFL1608Q4R7KTF -> XFL4015-471MEB; footprint Inductor_SMD:L_0603_1608Metric -> neg_footprints:Coilcraft-XFL4015
- Q3: LCSC C15127 -> (none)
- R4: value 0603WAF4992T5E -> RC0603FR-07732KL; LCSC C23184 -> (none)
- R5: value 0603WAF5601T5E -> CRCW0402100KFKED; footprint Resistor_SMD:R_0603_1608Metric -> Resistor_SMD:R_0402_1005Metric; LCSC C23189 -> (none)
- R6: value 0603WAF1003T5E -> CRCW0402316KFKED; footprint Resistor_SMD:R_0603_1608Metric -> Resistor_SMD:R_0402_1005Metric
- R7: value 0603WAF1802T5E -> CRCW0402100KFKED; footprint Resistor_SMD:R_0603_1608Metric -> Resistor_SMD:R_0402_1005Metric
- U2: value 74HC595 -> 74HC595D,112
- U3: value TLV61070ADBV -> TPS61023DRLR; footprint Package_TO_SOT_SMD:SOT-23-6 -> Package_TO_SOT_SMD:SOT-563; symbol Regulator_Switching:TLV61070ADBV -> neg_symbols:TPS61023DRLR; Digi-Key Part Number (none) -> 296-TPS61023DRLRCT-ND; LCSC C6881375 -> (none); Manufacturer (none) -> Texas Instruments; Manufacturer Part Number (none) -> TPS61023DRLR
- U4: value TLV61070ADBV -> TPS61021ADSGR; footprint Package_TO_SOT_SMD:SOT-23-6 -> neg_footprints:S-PWSON-N8; symbol Regulator_Switching:TLV61070ADBV -> neg_symbols:TPS61021ADSGR; Field5 (none) -> WFDFN-8 Texas Instruments; Field6 (none) -> None; Field7 (none) -> 3-A Boost Converter with 0.5-V Ultra Low Input Voltage 8-WS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; Field8 (none) -> Texas Instruments; Field9 (none) -> Unavailable
Connections:
- net BAT+: now also JP2.1 (A), JP3.1 (A), JP5.2 (B), SW3.1 (A); no longer JP1.2 (B)
- net BAT-: now also JP1.1 (A), U6.1 (VIN); no longer BT1.2 (-), BT2.2 (-), C3.2, C4.2, R7.2, SW3.1 (A), U4.2 (GND)
- net GND: now also SW3.3 (C), U3.4 (GND), U6.2 (GND), U6.5 (ST); no longer U3.2 (GND)
- net LED_VCC: now also Q3.3 (D)
- net at U4.1 (AGND): now also BT1.2 (-), BT2.2 (-), C3.2, C4.2, R7.2, U4.9 (PGND), Q1.2 (S); no longer L2.2
- net at C3.1, JP4.1 (A), L2.1: now also U4.5 (EN), U4.8 (VIN); no longer U4.3 (EN), U4.6 (V_{IN})
- net at R6.2, R7.1: now also U4.2 (FB), C5.2; no longer U4.4 (V_{FB})
- net at C4.1, JP5.1 (A), R6.1: now also U4.3 (VOUT), U4.4 (VOUT), C5.1; no longer U4.5 (V_{OUT})
- net at C2.1, JP16.1 (A), R4.1: now also U3.6 (V_{OUT}); no longer U3.5 (V_{OUT})
- net at SW3.2 (B): now also Q1.1 (G), Q2.1 (G); no longer Q3.1 (G)
- net at Q3.2 (S): now also JP14.2 (B)
- net at C1.1, JP15.2 (B), L1.1: now also U3.3 (V_{IN}); no longer U3.6 (V_{IN})
- net at L1.2: now also U3.5 (SW); no longer U3.1 (SW)
- net at SW4.2 (B): now also Q3.1 (G), U3.2 (EN); no longer U3.3 (EN)
- net at R4.2, R5.1: now also U3.1 (FB); no longer U3.4 (V_{FB})
- net LED_POWER renamed LED_CUTOFF
- new net: L2.2, U4.6 (SW), U4.7 (SW)
- new net: Q1.3 (D), Q2.3 (D)
- new net: JP1.2 (B), Q2.2 (S), U6.3 (~{CE}), U6.6 (VOUT)
Other:
- moved on the sheet: BT1, BT2, C3, C4, JP2, JP3, JP4, JP5, L2, R6, R7, U3
