File: negL/pcb_R/pcb_R.kicad_sch (KiCad schematic)
At the start: 149 parts, among them IC1 SN74LVC4245APWR, J1 MJ-4PP-9, J2 FH-1x4SG/RH, J3 XA-3-2-7P, Q1 AO3400A, Q2 AO3400A, Q3 AO3401A, SW1 TVBP06-B043CB-B, SW2 EVQWGD001_EC12, SW3 SS-12D00G3, SW4 SS-12D00G3, U1 nice_nano, U2 74HC595D,112, U3 TPS61023DRLR, U4 TPS61021ADSGR, U6 LM66100DCKR

Commit message: v0.1 rc
Parts:
- removed C2: C3216X5R1A226M160AC, Capacitor_SMD:C_1206_3216Metric, symbol Device:C
- removed IC1: SN74LVC4245APWR, Package_SO:TSSOP-24_4.4x7.8mm_P0.65mm, symbol neg_symbols:SN74LVC4245A
- removed Q1, Q2: AO3400A, Package_TO_SOT_SMD:SOT-23, symbol Transistor_FET:AO3400A
- removed Q3: AO3401A, Package_TO_SOT_SMD:SOT-23, symbol Transistor_FET:AO3401A
- added C4, C6, C7: CL10A226MP8NUNE, Capacitor_SMD:C_0603_1608Metric, symbol Device:C_Small
- added JP17, JP18: ~, Jumper:SolderJumper-2_P1.3mm_Open_Pad1.0x1.5mm, symbol Jumper:SolderJumper_2_Open
- added Q1, Q2: DMN1008UFDF-7, Package_DFN_QFN:Diodes_UDFN2020-6_Type-F, symbol neg_symbols:DMN1008UFDF
- added Q3: DMP1022UFDF-7, Package_DFN_QFN:Diodes_UDFN2020-6_Type-F, symbol PCM_marbastlib-various:DMP1022UFDF
- added U6: SN74LVC1T45DBVT, Package_TO_SOT_SMD:SOT-23-6, symbol Logic_LevelTranslator:SN74LVC1T45DBV
- C1: renamed from C3; LCSC C19702 -> (none)
- C3: renamed from C4; value GRM32ER61A107ME20L -> CL10A226MP8NUNE; footprint Capacitor_SMD:C_1210_3225Metric -> Capacitor_SMD:C_0603_1608Metric; symbol Device:C -> Device:C_Small; LCSC C59461 -> (none)
- C5: renamed from C1; value C1608X5R1A225K080AC -> GRM21BR61A226ME44L; footprint Capacitor_SMD:C_0603_1608Metric -> Capacitor_SMD:C_0805_2012Metric
- CH1, CH2: LCSC C5333465 -> (none)
- D1, D10, D11, D12, D13, D14, D15, D16, D17, D18, D19, D2, D20, D21, D22, D23, D24, D25, D26, D27, D28, D29, D3, D30, D31, D4, D5, D6, D7, D8, D9: LCSC C7420318 -> (none)
- L2: LCSC C1034 -> (none)
- LED1, LED10, LED11, LED12, LED13, LED14, LED15, LED16, LED17, LED18, LED19, LED2, LED20, LED21, LED22, LED23, LED24, LED25, LED26, LED27, LED28, LED29, LED3, LED4, LED5, LED6, LED7, LED8, LED9: LCSC C5149201 -> (none)
- MX1, MX10, MX11, MX12, MX13, MX14, MX15, MX16, MX17, MX18, MX19, MX2, MX20, MX21, MX22, MX23, MX24, MX25, MX26, MX27, MX3, MX4, MX5, MX6, MX7, MX8, MX9: LCSC C2803348 -> (none)
- R1: renamed from R6; LCSC C25803 -> (none)
- R2: renamed from R7; LCSC C25810 -> (none)
- R3: LCSC C22935 -> (none)
- R4: value RC0603FR-07732KL -> RC0603FR-07619KL
- R6: renamed from R2; LCSC C23162 -> (none)
- R7: renamed from R1; LCSC C23162 -> (none)
- U2: value 74HC595D,112 -> 74HC595D,118; LCSC C5947 -> (none)
- U3: Digi-Key Part Number 296-TPS61023DRLRCT-ND -> (none); Manufacturer Texas Instruments -> (none); Manufacturer Part Number TPS61023DRLR -> (none)
- U4: LCSC C6881375 -> (none)
- renumbered C5 to C2, MT9 to MT10, MT10 to MT11, MT11 to MT12, MT12 to MT5, MT5 to MT6, MT6 to MT7, MT7 to MT8, MT8 to MT9, U6 to U5
Connections:
- net DISP_SCL: now also JP18.1 (A); no longer R7.2
- net DISP_SDA: now also JP17.1 (A); no longer R6.2
- net GND: now also JP12.2 (B), C6.2, C7.2, U6.2 (GND); no longer JP13.2 (B)
- net LED: now also U6.3 (A)
- net LED_VCC: now also Q3.1 (D), Q3.2 (D), Q3.5 (D), Q3.6 (D), Q3.7 (D), U6.6 (VCCB)
- net VCC: now also JP13.1 (A), U6.5 (DIR); no longer JP12.1 (A)
- net at BT1.2 (-), BT2.2 (-), C1.2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: now also C4.2, Q2.4 (S), Q2.8 (S)
- net at C2.1, C3.1, JP5.1 (A)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: now also C4.1
- net at SW3.2 (B): now also Q1.3 (G), Q2.3 (G)
- net at JP16.1 (A), R4.1, U3.6 (V_{OUT}): now also C6.1, C7.1
- net at JP14.2 (B): now also Q3.4 (S), Q3.8 (S)
- net at SW4.2 (B), U3.2 (EN): now also Q3.3 (G)
- net at JP1.2 (B), U5.3 (~{CE}), U5.6 (VOUT): now also Q1.4 (S), Q1.8 (S)
- net at JP11.2 (B), LED1.3 (DIN): now also U6.4 (B)
- new net: JP12.1 (A), JP13.2 (B), U6.1 (VCCA)
- new net: JP18.2 (B), R7.2
- new net: JP17.2 (B), R6.2
- new net: Q1.1 (D), Q1.2 (D), Q1.5 (D), Q1.6 (D), Q1.7 (D), Q2.1 (D), Q2.2 (D), Q2.5 (D), Q2.6 (D), Q2.7 (D)
- no-connect marks 19 -> 5
Other:
- moved on the sheet: C3, J2, MT10, MT11, MT12, MT5, MT6, MT7, MT8, MT9, R6, R7

Commit message: v0.1
Parts:
- L1: value XFL4020-102MEB -> XAL4020-102MEC
Changed lines of the file:
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@@
 			)
 		)
-		(property "Value" "XFL4020-102MEB"
+		(property "Value" "XAL4020-102MEC"
 			(at 343.9595 251.0249 0)
 			(effects

Commit message: fix: update sch
Connections:
- net GND: no longer SW3.3 (C)
- net at BT1.2 (-), BT2.2 (-), C1.2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: now also SW3.3 (C)
Changed lines of the file:
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@@
 	)
 	(junction
+		(at 203.2 100.33)
+		(diameter 0)
+		(color 0 0 0 0)
+	)
+	(junction
 		(at 144.78 265.43)
 		(diameter 0)
@@
 	(wire
 		(pts
+			(xy 204.47 114.3) (xy 218.44 114.3)
+		)
+		(stroke
+			(width 0)
+			(type default)
+		)
+	)
+	(wire
+		(pts
 			(xy 375.92 128.27) (xy 375.92 110.49)
 		)
@@
 	(wire
 		(pts
+			(xy 218.44 114.3) (xy 218.44 100.33)
+		)
+		(stroke
+			(width 0)
+			(type default)
+		)
+	)
+	(wire
+		(pts
 			(xy 69.85 224.79) (xy 60.96 224.79)
 		)
@@
 	(wire
 		(pts
+			(xy 218.44 100.33) (xy 203.2 100.33)
+		)
+		(stroke
+			(width 0)
+			(type default)
+		)
+	)
+	(wire
+		(pts
 			(xy 160.02 247.65) (xy 160.02 265.43)
 		)
@@
 					(unit 1)
 				)
-			)
-		)
-	)
-	(symbol
-		(lib_id "power:GND")
-		(at 204.47 114.3 0)
-		(unit 1)
-		(exclude_from_sim no)
-		(in_bom yes)
-		(on_board yes)
-		(dnp no)
-		(fields_autoplaced yes)
-		(property "Reference" "#PWR037"
-			(at 204.47 120.65 0)
-			(effects
-				(font
-					(size 1.27 1.27)
-				)
-				(hide yes)
-			)
-		)
-		(property "Value" "GND"
-			(at 204.47 119.38 0)
-			(effects
-				(font
-					(size 1.27 1.27)
-				)
-			)
-		)
-		(property "Footprint" ""
-			(at 204.47 114.3 0)
-			(effects
-				(font
-					(size 1.27 1.27)
-				)
-				(hide yes)
-			)
-		)
-		(property "Datasheet" ""
-			(at 204.47 114.3 0)
-			(effects
-				(font
-					(size 1.27 1.27)
-				)
-				(hide yes)
-			)
-		)
-		(property "Description" "Power symbol creates a global label with name \"GND\" , ground"
-			(at 204.47 114.3 0)
-			(effects
-				(font
-					(size 1.27 1.27)
-				)
-				(hide yes)
-			)
-		)
-		(pin "1"
-		)
-		(instances
-			(project ""
-				(path "/9ab7ca09-b2ea-4853-bd3f-96554febaf98"
-					(reference "#PWR037")
-					(unit 1)
-				)
