File: negL/pcb_R/pcb_R.kicad_pcb (KiCad board)
At the start: 2 copper layers, 163 x 113.5 mm, 141 parts, among them IC1 SN74LVC4245A, J1 MJ-4PP-9, J2 FH-1x4SG/RH, J3 XA-3-2-7P, Q1 AO3400A, SW1 TVBP06-B043CB-B, SW2 EVQWGD001, SW3 SS-12D00G3, SW4 SS-12D00G3, U1 nice_nano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

Commit message: update
Parts:
- D31: value SS12 -> SS14
- moved JP3 22.6 mm to (83.3, 51.5)
- turned D31 to 180 degrees
Connections:
- BT2 pad 1: BAT+ -> Net-(BT2-+)
- C4 pad 1: Net-(D31-K) -> Net-(BT2-+)
- D31 pad 1: Net-(D31-K) -> BAT+
- D31 pad 2: BAT+ -> Net-(BT2-+)
- JP1 pad 1: BAT+ -> Net-(BT2-+)
- JP3 pad 1: Net-(D31-K) -> Net-(BT2-+)
- R6 pad 1: Net-(D31-K) -> Net-(BT2-+)
- SW3 pad 1: BAT+ -> Net-(BT2-+)
- U4 pad 5: Net-(D31-K) -> Net-(BT2-+)
Routing:
- net Net-(BT2-+): track 0.00 -> 40.2 mm, vias 0 -> 1
- net BAT+: track 45.1 -> 12.3 mm, vias 0 -> 1
- net Net-(D31-K): track 29.9 -> 0.00 mm, vias 2 -> 0

Commit message: update
Parts:
- added D32: 1N4148W, Diode_SMD:D_SOD-123, B.Cu at (84.0, 84.8)
Connections:
- JP4 pad 2: ROW3 -> Net-(D32-A)
Routing:
- net ROW3: track 169.6 -> 166.3 mm
- net Net-(D32-A): track 0.00 -> 2.73 mm

Commit message: update
Parts:
- removed JP10: LED switch input, Jumper:SolderJumper-2_P1.3mm_Open_Pad1.0x1.5mm
- added Q2: AO3401A, Package_TO_SOT_SMD:SOT-23, B.Cu at (77.4, 51.5)
- added Q3: AO3401A, Package_TO_SOT_SMD:SOT-23, B.Cu at (72.9, 52.2)
- MT1, MT10, MT11, MT2, MT3, MT4, MT5, MT6, MT7, MT8, MT9: value M2_SPACER -> MountingHole
- Q1: value AO3400A -> AO3401A
- SW2: value EVQWGD001 -> EVQWGD001_EC12
- moved Q1 32.0 mm to (73.8, 86.9)
- moved SW3 2.38 mm to (75.0, 48.8), turned to 0 degrees
- moved JP11 1.68 mm to (77.4, 86.9), turned to -90 degrees
- moved L2 1.62 mm to (76.4, 55.7)
- moved C3 1.53 mm to (76.4, 54.2)
Connections:
- BT1 pad 2: Net-(BT1--) -> BAT-
- BT2 pad 2: Net-(BT1--) -> BAT-
- C3 pad 2: Net-(BT1--) -> BAT-
- C4 pad 2: Net-(BT1--) -> BAT-
- D31 pad 2: Net-(BT2-+) -> Net-(D31-A)
- JP11 pad 1: Net-(JP11-A) -> VCC
- JP11 pad 2: LED_VCC -> Net-(JP11-B)
- JP3 pad 1: Net-(BT2-+) -> Net-(D31-A)
- Q1 pad 2: Net-(BT1--) -> Net-(JP11-B)
- Q1 pad 3: BAT- -> LED_VCC
- R3 pad 1: Net-(JP10-A) -> LED_POWER
- R7 pad 2: Net-(BT1--) -> BAT-
- SW2 pad MP: (no net) -> unconnected-(SW2-PadMP)_1
- SW3 pad 1: Net-(BT2-+) -> BAT-
- SW3 pad 2: Net-(Q1-G) -> Net-(Q2-G)
- SW3 pad 3: Net-(BT1--) -> Net-(BT2-+)
- SW4 pad 2: Net-(JP11-A) -> Net-(Q1-G)
- SW4 pad 3: Net-(JP10-A) -> LED_POWER
- U3 pad 3: Net-(JP11-A) -> Net-(Q1-G)
- U4 pad 2: Net-(BT1--) -> BAT-
Routing:
- net Net-(BT1--): track 95.8 -> 0.00 mm, vias 2 -> 0
- net BAT-: track 45.6 -> 132.0 mm, vias 0 -> 3
- net Net-(JP11-A): track 47.8 -> 0.00 mm, vias 4 -> 0
- net Net-(Q1-G): track 3.50 -> 49.0 mm, vias 1 -> 4
- net LED_POWER: track 47.4 -> 58.5 mm
- net Net-(BT2-+): track 40.2 -> 50.4 mm, vias 1 -> 0
- net Net-(JP10-A): track 9.80 -> 0.00 mm
- net Net-(D31-A): track 0.00 -> 9.15 mm
- net Net-(Q2-G): track 0.00 -> 6.80 mm
- net VCC: track 354.5 -> 361.1 mm, vias 6 -> 7
- net Net-(Q2-S): track 0.00 -> 4.80 mm
- net LED_VCC: track 701.2 -> 697.4 mm
- net Net-(JP11-B): track 0.00 -> 2.76 mm
- net Net-(U4-SW): track 3.77 -> 1.78 mm
- net ROW4: track 247.2 -> 249.2 mm
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
Commit message: update
Parts:
- removed the JP9 at (76.2, 71.4)
- added JP10: LED_VCC 5V, Jumper:SolderJumper-2_P1.3mm_Open_Pad1.0x1.5mm, B.Cu at (78.0, 75.9)
- SW2: footprint neg_footprints:EVQWGD001_EC12 -> neg_footprints:choc_encoder
- moved MT5 18.3 mm to (90.5, 122.6)
- moved C3 14.2 mm to (79.3, 68.1), turned to -90 degrees
- moved J1 13.4 mm to (66.7, 115.5), turned to -90 degrees
- moved Q3 12.7 mm to (83.3, 59.5)
- moved D26 12.2 mm to (100.0, 139.3)
- moved C4 11.1 mm to (75.9, 73.1)
- moved U4 10.8 mm to (76.2, 69.1)
- moved L2 10.7 mm to (76.1, 66.4)
- moved R6 10.6 mm to (73.1, 69.1)
- moved R7 10.6 mm to (76.0, 71.5)
- moved JP1 9.56 mm to (85.7, 68.8)
- moved MT4 9.29 mm to (80.4, 138.7)
- moved SW1 8.46 mm to (64.6, 125.0)
- moved Q2 8.37 mm to (75.0, 59.5)
- moved JP6 8.04 mm to (85.7, 75.5), turned to 90 degrees
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- renumbered D32 to D31, D31 to D32, JP12 to JP11, JP13 to JP12, JP11 to JP9
Routing:
- net Net-(D30-A): track 20.3 -> 57.7 mm
- net COL0: track 115.1 -> 139.6 mm
- net Net-(JP5-A): track 53.2 -> 69.4 mm, vias 1 -> 2
- net Net-(Q1-G): track 49.0 -> 34.3 mm, vias 4 -> 2
- net BAT-: track 132.0 -> 119.9 mm, vias 3 -> 1
- net Net-(JP6-A): track 55.5 -> 66.4 mm, vias 1 -> 2
- net Net-(D32-A): track 9.15 -> 18.1 mm
- net VCC: track 361.1 -> 353.0 mm, vias 7 -> 8
- net RESET: track 80.7 -> 87.3 mm
- net DATA_TX: track 49.5 -> 55.8 mm
- net Net-(BT2-+): track 50.4 -> 56.6 mm
- net Net-(Q2-G): track 6.80 -> 12.4 mm, vias 0 -> 1
- net Net-(JP2-A): track 20.4 -> 15.0 mm
- net Net-(LED3-DOUT): track 89.0 -> 94.0 mm
- net Net-(LED1-DOUT): track 19.7 -> 24.7 mm
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Other:
- board size 163 x 113.5 mm -> 168.4 x 115.6 mm

Commit message: update
Parts:
- moved SW1 1.68 mm to (63.4, 126.2)
- moved J1 1.19 mm to (65.5, 115.5)
Routing:
- net GND: track 839.1 -> 842.0 mm
- net RESET: track 87.3 -> 88.9 mm
- net VCC: track 353.0 -> 354.2 mm
- net Net-(JP6-A): track 66.4 -> 67.6 mm
- net Net-(JP5-A): track 69.4 -> 70.6 mm
- net COL0: track 139.6 -> 140.8 mm
Other:
- outline, holes or cut-outs redrawn
