File: negL/ball_breakout_compat/ball_breakout.kicad_sch (KiCad schematic)
At the start: 19 parts, among them J1 XA-3-2-7P Contact, U1 PAW3395, U4 SK6615C

Commit message: update
Parts:
- added C8, C9: CL10A106KP8NNNC, Capacitor_SMD:C_0603_1608Metric, symbol Device:C
- added D1, D2, D3: BZT52C3V3S, Diode_SMD:D_SOD-323, symbol Device:D_Zener
- added L1: SDFL2012Q1R0KTF, Inductor_SMD:L_0805_2012Metric, symbol Device:L
- added R3: 0603WAF5603T5E, Resistor_SMD:R_0603_1608Metric, symbol Device:R
- added R4: 0603WAF1303T5E, Resistor_SMD:R_0603_1608Metric, symbol Device:R
- added U3: SK6615C, Package_TO_SOT_SMD:SOT-23-5, symbol neg_symbols:SK6615CS5
- JP1: symbol Jumper:SolderJumper_2_Open -> Jumper:SolderJumper_2_Bridged
Connections:
- net 3V3: now also C9.1, L1.2, R3.1; no longer C10.1, J1.4 (Pin_4), U4.1 (EN), U4.4 (VIN)
- net GND: now also C8.2, C9.2, D1.2 (A), D2.2 (A), D3.2 (A), R4.2, U3.2 (GND)
- net MOSI: now also D3.1 (K)
- net NCS: now also D2.1 (K)
- net SCLK: now also D1.1 (K)
- new net: R3.2, R4.1, U3.5 (FB)
- new net: L1.1, U3.3 (SW)
- new net VCC: C10.1, C8.1, J1.4 (Pin_4), U3.1 (EN), U3.4 (VIN), U4.1 (EN), U4.4 (VIN)
