File: negL/bottom_R/bottom_R.kicad_pcb (KiCad board)
At the start: 2 copper layers, 162.7 x 113.5 mm, 9 parts

Commit message: add bottom
Parts:
- removed MT1: M2_Bottom, neg_footprints:M2_Bottom
- added MT12: MountingHole, MountingHole:MountingHole_2.7mm_M2.5, F.Cu at (199.7, 135.6)
- added MT2: MountingHole, MountingHole:MountingHole_2.7mm_M2.5, F.Cu at (87.7, 90.3)
- added MT3: MountingHole, MountingHole:MountingHole_2.7mm_M2.5, F.Cu at (102.0, 90.3)
- added REF**: M1.7_bottom, neg_footprints:M1.7_bottom, F.Cu at (156.9, 139.8)
- added REF**: M1.7_bottom, neg_footprints:M1.7_bottom, F.Cu at (156.9, 123.8)
- MT10, MT11, MT4, MT5, MT6, MT7, MT8, MT9: value M2_Bottom -> MountingHole; footprint neg_footprints:M2_Bottom -> MountingHole:MountingHole_2.7mm_M2.5
- moved MT6 88.4 mm to (97.3, 129.6)
- moved MT8 78.0 mm to (123.5, 108.2)
- moved MT10 74.7 mm to (161.6, 108.2)
- moved MT11 62.3 mm to (199.7, 53.4)
- moved MT9 44.2 mm to (161.6, 48.6)
- moved MT7 36.5 mm to (123.5, 57.0)
- moved MT5 32.3 mm to (85.4, 118.9)
- moved MT4 20.3 mm to (74.6, 128.4)
Other:
- board size 162.7 x 113.5 mm -> 168.4 x 117.5 mm
- board text added: "MX_SK6812MINI-E"
- board text removed: "Designed by nazo6, 2024"
- board text removed: "negL"
- board text removed: "test1"

Commit message: update
Parts:
- removed the REF** at (156.9, 139.8)
- removed the REF** at (156.9, 123.8)
- added MT3: MountingHole, MountingHole:MountingHole_2.7mm_M2.5, F.Cu at (94.9, 47.4)
- added REF**: M1.7_bottom, neg_footprints:M1.7_bottom, F.Cu at (155.3, 140.5)
- added REF**: M1.7_bottom, neg_footprints:M1.7_bottom, F.Cu at (155.3, 124.8)
Other:
- outline, holes or cut-outs redrawn
