File: negL/pcb_L/pcb_L.kicad_pcb (KiCad board)
At the start: 2 copper layers, 168.4 x 117.5 mm, 161 parts, among them J1 MJ-4PP-9, J2 FH-1x4SG/RH, Q1 DMN1008UFDF-7, Q2 DMN1008UFDF-7, Q3 DMP1022UFDF-7, SW1 TVBP06-B043CB-B, SW2 EVQWGD001_EC12, SW3 SS-12D00G3, SW4 SS-12D00G3, U1 nice_nano, U2 74HC595D,118, U3 TPS61023DRLR, U4 TPS61021ADSGR, U5 LM66100DCKR, U6 SN74LVC1T45DBVT

Commit message: pcb-l update
Parts:
- removed Q1: DMN1008UFDF-7, Package_DFN_QFN:Diodes_UDFN2020-6_Type-F
- L1: value XAL4020-102MEC -> XFL4015-471MEB
- L2: footprint neg_footprints:Coilcraft-XFL4015 -> Inductor_SMD:L_Coilcraft_XxL4020
- moved JP17 240.3 mm to (197.3, 80.4), turned to -90 degrees
- moved R6 239.2 mm to (197.3, 84.5), turned to 90 degrees
- moved R7 232.2 mm to (193.9, 84.6), turned to 90 degrees
- moved JP18 232.2 mm to (194.0, 80.4), turned to -90 degrees
- moved BT1 221.5 mm to (199.9, 62.3)
- moved BT2 221.5 mm to (197.0, 55.3)
- moved C2 221.5 mm to (203.4, 90.2)
- moved C3 221.5 mm to (203.4, 91.8)
- moved CH2 221.5 mm to (167.7, 134.7)
- moved CH3 221.5 mm to (146.3, 133.5)
- moved D1 221.5 mm to (161.8, 60.9)
- moved D12 221.5 mm to (66.5, 68.0)
- moved D13 221.5 mm to (161.8, 81.1)
- moved D14 221.5 mm to (142.7, 81.1)
- moved D15 221.5 mm to (123.7, 81.1)
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Connections:
- J1 pad R1: Net-(JP7-A) -> Net-(JP17-A)
- JP17 pad 1: DISP_SDA -> Net-(JP17-A)
- JP18 pad 1: DISP_SCL -> Net-(JP10-A)
- JP7 pad 1: Net-(JP7-A) -> Net-(JP17-A)
- JP9 pad 1: Net-(JP7-A) -> Net-(JP17-A)
- Q2 pad 1: Net-(Q1-D-Pad1) -> Net-(JP1-B)
- Q2 pad 2: Net-(Q1-D-Pad1) -> Net-(JP1-B)
- Q2 pad 5: Net-(Q1-D-Pad1) -> Net-(JP1-B)
- Q2 pad 6: Net-(Q1-D-Pad1) -> Net-(JP1-B)
- Q2 pad 7: Net-(Q1-D-Pad1) -> Net-(JP1-B)
Routing:
- net Net-(JP17-A): track 0.00 -> 67.2 mm, vias 0 -> 1
- net Net-(JP7-A): track 64.7 -> 0.00 mm, vias 1 -> 0
- net VCC: track 200.4 -> 220.1 mm, vias 7 -> 9
- net Net-(Q1-D-Pad1): track 15.0 -> 0.00 mm
- net Net-(JP1-B): track 27.6 -> 35.0 mm
- net DISP_SCL: track 26.8 -> 22.1 mm
- net DISP_SDA: track 32.9 -> 29.0 mm
- net COL0: track 119.1 -> 116.7 mm
- net Net-(Q2-G): track 9.63 -> 7.77 mm
- net Net-(BT1--): track 101.1 -> 99.7 mm
- net Net-(JP17-B): track 3.94 -> 2.65 mm
- net LED_CUTOFF: track 48.7 -> 47.6 mm
- net Net-(JP18-B): track 3.64 -> 2.80 mm
- net Net-(JP10-A): track 57.9 -> 58.4 mm
Other:
- outline, holes or cut-outs redrawn

Commit message: update
Parts:
- removed C5: GRM21BR61A226ME44L, Capacitor_SMD:C_0805_2012Metric
- removed C6, C7: CL10A226MP8NUNE, Capacitor_SMD:C_0603_1608Metric
- removed JP12, JP13, JP15, JP16: ~, Jumper:SolderJumper-2_P1.3mm_Open_Pad1.0x1.5mm
- removed L1: XFL4015-471MEB, Inductor_SMD:L_Coilcraft_XxL4020
- removed R4: RC0603FR-07619KL, Resistor_SMD:R_0603_1608Metric
- removed R5: CRCW0402100KFKED, Resistor_SMD:R_0402_1005Metric
- removed U3: TPS61023DRLR, Package_TO_SOT_SMD:SOT-563
- removed U6: SN74LVC1T45DBVT, Package_TO_SOT_SMD:SOT-23-6
Routing:
- net GND: track 803.6 -> 774.4 mm, vias 14 -> 43
- net LED_VCC: track 718.1 -> 696.4 mm, vias 15 -> 13
- net VCC: track 220.1 -> 205.8 mm, vias 9 -> 8
- net Net-(JP16-A): track 13.4 -> 0.00 mm
- net Net-(JP15-B): track 13.3 -> 0.00 mm
- net Net-(JP12-A): track 12.4 -> 0.00 mm
- net Net-(JP11-B): track 31.0 -> 22.0 mm, vias 2 -> 0
- net LED: track 62.8 -> 56.4 mm
- net Net-(U3-FB): track 5.79 -> 0.00 mm
- net Net-(U3-SW): track 5.15 -> 0.00 mm, vias 2 -> 0
- net Net-(Q3-G): track 38.9 -> 38.4 mm, vias 4 -> 2
- net (no net): vias 0 -> 1

Commit message: update pcb_L
Parts:
- added JP13: ~, Jumper:SolderJumper-2_P1.3mm_Open_Pad1.0x1.5mm, B.Cu at (181.6, 90.5)
- added JP14: ~, Jumper:SolderJumper-2_P1.3mm_Open_Pad1.0x1.5mm, B.Cu at (178.2, 90.5)
- added R4: 0603WAF4701T5E, Resistor_SMD:R_0603_1608Metric, B.Cu at (181.6, 94.9)
- added R5: 0603WAF4701T5E, Resistor_SMD:R_0603_1608Metric, B.Cu at (178.2, 95.0)
- renumbered JP17 to JP11, JP18 to JP12, JP11 to JP15, JP14 to JP16, L2 to L1, Q2 to Q1, Q3 to Q2, U4 to U2, U5 to U3, U2 to U4
Connections:
- SW2 pad C: VCC -> GND
Routing:
- net VCC: track 205.8 -> 124.2 mm, vias 8 -> 7
- net GND: track 774.4 -> 816.5 mm, vias 43 -> 61
- net DISP_SDA: track 29.0 -> 35.3 mm
- net DISP_SCL: track 22.1 -> 28.1 mm
- net Net-(JP14-B): track 0.00 -> 3.10 mm
- net Net-(JP13-B): track 0.00 -> 2.98 mm
- net (no net): vias 1 -> 0
Other:
- board text added: "B+"
- board text added: "B-"
- board text added: "CNCS"
- board text added: "DSCL"
- board text added: "DSDA"
- board text added: "ENCA"
- board text added: "ENCB"
- board text added: "GND"
- board text added: "LCOF"
- board text added: "LED"
- board text added: "MISO"
- board text added: "MOSI"
- board text added: "ROW0"
- board text added: "ROW1"
- board text added: "ROW2"
- board text added: "ROW3"
- board text added: "ROW4"
- board text added: "RST"
- board text added: "RX"
- board text added: "SCK"
- board text added: "TX"
- board text added: "VCC"
