File: negL/pcb_L/pcb_L.kicad_pcb (KiCad board)
At the start: 2 copper layers, 168.4 x 117.5 mm, 152 parts, among them J1 MJ-4PP-9, J2 FH-1x4SG/RH, Q1 DMN1008UFDF-7, Q2 DMP1022UFDF-7, SW1 TVBP06-B043CB-B, SW2 EVQWGD001_EC12, SW3 SS-12D00G3, SW4 SS-12D00G3, U1 nice_nano, U2 TPS61021ADSGR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

Commit message: update
Parts:
- moved MT7 8.49 mm to (114.1, 53.6)
