File: negL/pcb_L/pcb_L.kicad_sch (KiCad schematic)
At the start: 161 parts, among them J1 MJ-4PP-9, J2 FH-1x4SG/RH, Q1 DMN1008UFDF-7, Q2 DMN1008UFDF-7, Q3 DMP1022UFDF-7, SW1 TVBP06-B043CB-B, SW2 EVQWGD001_EC12, SW3 SS-12D00G3, SW4 SS-12D00G3, U1 nice_nano, U2 74HC595D,118, U3 TPS61023DRLR, U4 TPS61021ADSGR, U5 LM66100DCKR, U6 SN74LVC1T45DBVT

Commit message: pcb-l update
Parts:
- removed Q1: DMN1008UFDF-7, Package_DFN_QFN:Diodes_UDFN2020-6_Type-F, symbol neg_symbols:DMN1008UFDF
- C1: LCSC (none) -> C19702
- CH1, CH2, CH3: LCSC (none) -> C5333465
- D1, D10, D11, D12, D13, D14, D15, D16, D17, D18, D19, D2, D20, D21, D22, D23, D24, D25, D26, D27, D28, D29, D3, D30, D31, D32, D33, D34, D4, D5, D6, D7, D8, D9: LCSC (none) -> C7420318
- L1: value XAL4020-102MEC -> XFL4015-471MEB
- L2: footprint neg_footprints:Coilcraft-XFL4015 -> Inductor_SMD:L_Coilcraft_XxL4020
- LED1, LED10, LED11, LED12, LED13, LED14, LED15, LED16, LED17, LED18, LED19, LED2, LED20, LED21, LED22, LED23, LED24, LED25, LED26, LED27, LED28, LED29, LED3, LED30, LED31, LED32, LED4, LED5, LED6, LED7, LED8, LED9: LCSC (none) -> C5149201
- MX1, MX10, MX11, MX12, MX13, MX14, MX15, MX16, MX17, MX18, MX19, MX2, MX20, MX21, MX22, MX23, MX24, MX25, MX26, MX27, MX28, MX29, MX3, MX4, MX5, MX6, MX7, MX8, MX9: LCSC (none) -> C2803348
- R1: LCSC (none) -> C25803
- R2: LCSC (none) -> C25810
- R3: LCSC (none) -> C22935
- U2: LCSC (none) -> C5947
- U4: LCSC (none) -> C6881375
Connections:
- net DISP_SCL: no longer JP18.1 (A)
- net DISP_SDA: no longer JP17.1 (A)
- net at J1.R1, JP7.1 (A), JP9.1 (A): now also JP17.1 (A)
- net at JP1.2 (B), U5.3 (~{CE}), U5.6 (VOUT): now also Q2.1 (D), Q2.2 (D), Q2.5 (D), Q2.6 (D), Q2.7 (D)
- net at J1.T, JP10.1 (A), JP8.1 (A): now also JP18.1 (A)
- no-connect marks 6 -> 7
Other:
- moved on the sheet: JP10, JP7, JP8, JP9, Q2, SW3

Commit message: update
Parts:
- removed C5: GRM21BR61A226ME44L, Capacitor_SMD:C_0805_2012Metric, symbol Device:C
- removed C6, C7: CL10A226MP8NUNE, Capacitor_SMD:C_0603_1608Metric, symbol Device:C_Small
- removed JP12, JP13, JP15, JP16: ~, Jumper:SolderJumper-2_P1.3mm_Open_Pad1.0x1.5mm, symbol Jumper:SolderJumper_2_Open
- removed L1: XFL4015-471MEB, Inductor_SMD:L_Coilcraft_XxL4020, symbol Device:L
- removed R4: RC0603FR-07619KL, Resistor_SMD:R_0603_1608Metric, symbol Device:R
- removed R5: CRCW0402100KFKED, Resistor_SMD:R_0402_1005Metric, symbol Device:R
- removed U3: TPS61023DRLR, Package_TO_SOT_SMD:SOT-563, symbol neg_symbols:TPS61023DRLR
- removed U6: SN74LVC1T45DBVT, Package_TO_SOT_SMD:SOT-23-6, symbol Logic_LevelTranslator:SN74LVC1T45DBV
- C1: LCSC C19702 -> (none)
- CH1, CH2, CH3: LCSC C5333465 -> (none); now left out of the parts list
- D1, D10, D11, D12, D13, D14, D15, D16, D17, D18, D19, D2, D20, D21, D22, D23, D24, D25, D26, D27, D28, D29, D3, D30, D31, D32, D33, D34, D4, D5, D6, D7, D8, D9: LCSC C7420318 -> (none)
- LED1, LED10, LED11, LED12, LED13, LED14, LED15, LED16, LED17, LED18, LED19, LED2, LED20, LED21, LED22, LED23, LED24, LED25, LED26, LED27, LED28, LED29, LED3, LED30, LED31, LED32, LED4, LED5, LED6, LED7, LED8, LED9: LCSC C5149201 -> (none); now left out of the parts list
- MX1, MX10, MX11, MX12, MX13, MX14, MX15, MX16, MX17, MX18, MX19, MX2, MX20, MX21, MX22, MX23, MX24, MX25, MX26, MX27, MX28, MX29, MX3, MX4, MX5, MX6, MX7, MX8, MX9: LCSC C2803348 -> (none); now left out of the parts list
- R1: LCSC C25803 -> (none)
- R2: LCSC C25810 -> (none)
- R3: LCSC C22935 -> (none)
- SW2: now left out of the parts list
- U2: LCSC C5947 -> (none)
- U4: LCSC C6881375 -> (none)
Other:
- moved on the sheet: J2, JP11, JP14

Commit message: update pcb_L
Parts:
- added JP13, JP14: ~, Jumper:SolderJumper-2_P1.3mm_Open_Pad1.0x1.5mm, symbol Jumper:SolderJumper_2_Open
- added R4, R5: 0603WAF4701T5E, Resistor_SMD:R_0603_1608Metric, symbol Device:R
- renumbered JP17 to JP11, JP18 to JP12, JP11 to JP15, JP14 to JP16, L2 to L1, Q2 to Q1, Q3 to Q2, U4 to U2, U5 to U3, U2 to U4
Connections:
- net DISP_SCL: now also JP13.1 (A)
- net DISP_SDA: now also JP14.1 (A)
- net GND: now also SW2.C
- net VCC: now also R4.1, R5.1; no longer SW2.C
- new net: JP14.2 (B), R5.2
- new net: JP13.2 (B), R4.2
Other:
- moved on the sheet: J2
